File: template/EnvOpenPico.kicad_pcb (KiCad board)
At the start: 2 copper layers, 21.1 x 51.3 mm, 37 parts, among them J2 B3U-1000P, J3 2.54mm header 01x20, J4 2.54mm header 01x20, J5 Conn_01x03_Male, U1 SPX3819M5-L-3-3, U3 RP2040, X1 XO 32 12Mhz 3225 seiko

Commit message: nothing
Parts:
- FLASH1: value W25Q128JVPIQ -> W25Q16JVUXIQ
Connections:
- FLASH1 pad 9: (no net) -> Net-(FLASH1-Pad9)
- J4 pad 2: (no net) -> Net-(J4-Pad2)
- J4 pad 6: (no net) -> Net-(J4-Pad6)
- U1 pad 4: (no net) -> Net-(U1-Pad4)
- U3 pad 21: (no net) -> /XOUT
- U3 pad 35: (no net) -> /GPIO23
- U3 pad 36: (no net) -> /GPIO24
- U3 pad 41: (no net) -> /GPIO29_ADC3
- X1 pad 1: (no net) -> Net-(X1-Pad1)
- e1 pad 3: (no net) -> Net-(e1-Pad3)
- e1 pad 9: (no net) -> Net-(e1-Pad9)
